File: Training_Based.kicad_sch (KiCad schematic)
At the start: 0 parts

Commit message: update
Parts:
- added U (x6): (no value), symbol Mechanical:MountingHole_Pad
Connections:
- new net GND: U.1, U.1, U.1, U.1, U.1, U.1
Other:
- note added: "7 Segment 4 Digit TM1637"
- note added: "Buzzer (Operating Voltage 1-6V)"
- note added: "ESP32 38 PIN"
- note added: "LDR (10 mm)"
- note added: "PIR Sensor"
- note added: "Relay (coil = 5V)"
- note added: "Temp/Humid"
- note added: "Ultrasonic HC-SR04"
