File: Training_Based.kicad_sch (KiCad schematic)
At the start: 18 parts

Commit message: work in progress 650723.0501
Parts:
- removed TH: DHT11_Temperature_Humidity, symbol sensors:DHT11_Temperature_Humidity
- added BZ: Buzzer, symbol Device:Buzzer
- added D (x8): LED, symbol Device:LED
- added Q (x9): BC817, Package_TO_SOT_SMD:SOT-23, symbol Transistor_BJT:BC817
- added R (x18): R_Small, symbol Device:R_Small
- added TH: DHT22_Temperature_Humidity, symbol sensors:DHT22_Temperature_Humidity
- added U: esp32_38_pins-custom_library, esp32_lora_v2:esp32_devkitv4_38pin, symbol FP:esp32_38_pins-custom_library
Connections:
- net +5V: now also J.19 (Pin_19), J.19 (Pin_19), BZ.1 (-), D.2 (A), D.2 (A), D.2 (A), D.2 (A), D.2 (A), D.2 (A), D.2 (A), D.2 (A), U.19 (5V)
- net GND: now also J.1 (Pin_1), J.1 (Pin_1), J.14 (Pin_14), J.14 (Pin_14), J.7 (Pin_7), J.7 (Pin_7), Q.2 (E), Q.2 (E), Q.2 (E), Q.2 (E), Q.2 (E), Q.2 (E), Q.2 (E), Q.2 (E), Q.2 (E), U.14 (GND), U.32 (GND), U.38 (GND)
- net +3.3V: now reaches J.1 (Pin_1), J.1 (Pin_1)
- net +3.3V: now also U.1 (3.3V)
- net GPIO26: now reaches J.10 (Pin_10), J.10 (Pin_10)
- net GPIO26: now also U.10 (GPIO26)
- net GPIO27: now reaches J.11 (Pin_11), J.11 (Pin_11)
- net GPIO27: now also U.11 (GPIO27)
- net GPIO14: now reaches J.12 (Pin_12), J.12 (Pin_12)
- net GPIO14: now also U.12 (GPIO14)
- net GPIO12: now reaches J.13 (Pin_13), J.13 (Pin_13)
- net GPIO12: now also U.13 (GPIO12)
- net GPIO13: now reaches J.15 (Pin_15), J.15 (Pin_15)
- net GPIO13: now also U.15 (GPIO13)
- net GPIO9: now reaches J.16 (Pin_16), J.16 (Pin_16)
- net GPIO9: now also U.16 (GPIO9)
- net GPIO10: now reaches J.17 (Pin_17), J.17 (Pin_17)
- net GPIO10: now also U.17 (GPIO10)
- net GPIO11: now reaches J.18 (Pin_18), J.18 (Pin_18)
- net GPIO11: now also U.18 (GPIO11)
- net EN_RST: now reaches J.2 (Pin_2), J.2 (Pin_2)
- net EN_RST: now also U.2 (EN_RST)
- net GPI36: now reaches J.3 (Pin_3), J.3 (Pin_3)
- net GPI36: now also U.3 (GPI36)
- net GPI39: now reaches J.4 (Pin_4), J.4 (Pin_4)
- net GPI39: now also U.4 (GPI39)
- net GPI34: now reaches J.5 (Pin_5), J.5 (Pin_5)
- net GPI34: now also U.5 (GPI34)
- net GPI35: now reaches J.6 (Pin_6), J.6 (Pin_6)
- net GPI35: now also U.6 (GPI35)
- net GPIO32: now reaches J.7 (Pin_7), J.7 (Pin_7)
- net GPIO32: now also U.7 (GPIO32)
- net GPIO33: now reaches J.8 (Pin_8), J.8 (Pin_8)
- net GPIO33: now also U.8 (GPIO33)
- net GPIO25: now reaches J.9 (Pin_9), J.9 (Pin_9)
- net GPIO25: now also U.9 (GPIO25)
- net at Q.1 (B): now also R.2
- net GPIO5: now reaches J.10 (Pin_10), J.10 (Pin_10)
- net GPIO5: now also U.29 (GPIO5)
- net GPIO17: now reaches J.11 (Pin_11), J.11 (Pin_11)
- net GPIO17: now also U.28 (GPIO17)
- net GPIO16: now reaches J.12 (Pin_12), J.12 (Pin_12)
- net GPIO16: now also U.27 (GPIO16)
- net GPIO4: now reaches J.13 (Pin_13), J.13 (Pin_13)
- net GPIO4: now also U.26 (GPIO4)
- net GPIO0: now reaches J.14 (Pin_14), J.14 (Pin_14)
- net GPIO0: now also U.25 (GPIO0)
- net GPIO2: now reaches J.15 (Pin_15), J.15 (Pin_15)
- net GPIO2: now also U.24 (GPIO2)
- net GPIO15: now reaches J.16 (Pin_16), J.16 (Pin_16)
- net GPIO15: now also U.23 (GPIO15)
- net GPIO8: now reaches J.17 (Pin_17), J.17 (Pin_17)
- net GPIO8: now also U.22 (GPIO8)
- net GPIO7: now reaches J.18 (Pin_18), J.18 (Pin_18)
- net GPIO7: now also U.21 (GPIO7)
- net GPIO6: now reaches J.19 (Pin_19), J.19 (Pin_19)
- net GPIO6: now also U.20 (GPIO6)
- net GPIO23: now reaches J.2 (Pin_2), J.2 (Pin_2)
- net GPIO23: now also U.37 (GPIO23)
- net GPIO22: now reaches J.3 (Pin_3), J.3 (Pin_3)
- net GPIO22: now also U.36 (GPIO22)
- net GPIO1: now reaches J.4 (Pin_4), J.4 (Pin_4)
- net GPIO1: now also U.35 (GPIO1)
- net GPIO3: now reaches J.5 (Pin_5), J.5 (Pin_5)
- net GPIO3: now also U.34 (GPIO3)
- net GPIO21: now reaches J.6 (Pin_6), J.6 (Pin_6)
- net GPIO21: now also U.33 (GPIO21)
- net GPIO19: now reaches J.8 (Pin_8), J.8 (Pin_8)
- net GPIO19: now also U.31 (GPIO19)
- net GPIO18: now reaches J.9 (Pin_9), J.9 (Pin_9)
- net GPIO18: now also U.30 (GPIO18)
- new net: D.1 (K), R.1 (x8)
- new net: Q.1 (B), R.2 (x9)
- new net: Q.3 (C), R.2 (x8)
- new net: BZ.2 (+), Q.3 (C)
- new net BUZZER1: R.1
- new net BUZZER2: R.1
- new net LED1: R.1, R.1, R.1, R.1, R.1, R.1, R.1, R.1
Other:
- moved on the sheet: J, K

Commit message: WIP 6507230502
Parts:
- added D (x2): D, symbol Device:D
- added J: Conn_01x08, symbol Connector_Generic:Conn_01x08
- added Q (x2): BC817, Package_TO_SOT_SMD:SOT-23, symbol Transistor_BJT:BC817
- added R (x2): R_Small, symbol Device:R_Small
Connections:
- net +5V: now also K.A1, K.A1, D.1 (K), D.1 (K)
- net GND: now also Q.2 (E), Q.2 (E)
- net LED1: now also J.1 (Pin_1); no longer R.1, R.1, R.1, R.1, R.1, R.1, R.1
- net at K.A2: now also D.2 (A), Q.3 (C) (x2)
- new net: Q.1 (B), R.2 (x2)
- new net LED2: J.2 (Pin_2), R.1
- new net LED3: J.3 (Pin_3), R.1
- new net LED4: J.4 (Pin_4), R.1
- new net LED5: J.5 (Pin_5), R.1
- new net LED6: J.6 (Pin_6), R.1
- new net LED7: J.7 (Pin_7), R.1
- new net LED8: J.8 (Pin_8), R.1
- new net RELAY1: R.1
- new net RELAY2: R.1
Other:
- moved on the sheet: K

Commit message: Update Training_Based.kicad_sch
Parts:
- added J (x4): Conn_02x02_Row_Letter_Last, symbol Connector_Generic:Conn_02x02_Odd_Even
Connections:
- net +5V: now also TH.1 (VDD), U.1 (Vcc)
- net BUZZER1: now also J.1 (Pin_1), J.3 (Pin_3)
- net BUZZER2: now also J.2 (Pin_2), J.4 (Pin_4)
- net GND: now also TH.4 (GND), U.4 (Gnd)
- net RELAY1: now also J.1 (Pin_1), J.2 (Pin_2)
- net RELAY2: now also J.3 (Pin_3), J.4 (Pin_4)
- net Trig: now reaches U.2 (Trig)
- net Trig: now also J.3 (Pin_3), J.4 (Pin_4)
- net Echo: now reaches U.3 (Echo)
- net Echo: now also J.1 (Pin_1), J.2 (Pin_2)
- net DATA: now reaches TH.2 (DATA)
- net DATA: now also J.3 (Pin_3), J.4 (Pin_4)
- net at TH.3 (NULL): now also J.1 (Pin_1), J.2 (Pin_2)
Other:
- moved on the sheet: AFF, BZ, D, J, K, PIR, Q, R, TH, U
