File: Training_Based.kicad_sch (KiCad schematic)
At the start: 134 parts

Commit message: Update Training_Based.kicad_sch
Connections:
- net +3.3V: no longer J.1 (Pin_1), J.1 (Pin_1), U.1 (3.3V)
- new net +3.3V_ESP: J.1 (Pin_1), J.1 (Pin_1), U.1 (3.3V)
Changed lines of the file:
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@@
     (stroke (width 0) (type default))
   )
-  (wire (pts (xy 57.785 185.42) (xy 57.785 187.325))
-    (stroke (width 0) (type default))
-  )
   (wire (pts (xy 349.25 96.52) (xy 349.25 97.155))
     (stroke (width 0) (type default))
@@
     (effects (font (size 1.27 1.27)) (justify left bottom))
   )
-  (label "+3.3V" (at 33.02 187.325 0) (fields_autoplaced)
+  (label "+3.3V_ESP" (at 33.02 187.325 0) (fields_autoplaced)
     (effects (font (size 1.27 1.27)) (justify left bottom))
   )
@@
     (effects (font (size 1.27 1.27)) (justify left bottom))
   )
+  (label "+3.3V_ESP" (at 67.945 187.325 0) (fields_autoplaced)
+    (effects (font (size 1.27 1.27)) (justify right bottom))
+  )
   (label "S_D" (at 396.875 33.02 0) (fields_autoplaced)
     (effects (font (size 1.27 1.27)) (justify left bottom))
@@
     (effects (font (size 1.27 1.27)) (justify left bottom))
   )
-  (label "+3.3V" (at 59.69 187.325 0) (fields_autoplaced)
-    (effects (font (size 1.27 1.27)) (justify left bottom))
-  )
   (label "GPIO13" (at 33.02 222.885 0) (fields_autoplaced)
     (effects (font (size 1.27 1.27)) (justify left bottom))
@@
     (pin "1")
   )
-  (symbol (lib_id "power:+3.3V") (at 57.785 185.42 0) (unit 1)
-    (in_bom yes) (on_board yes) (fields_autoplaced)
-    (default_instance (reference "#PWR") (unit 1) (value "+3.3V") (footprint ""))
-    (property "Reference" "#PWR" (id 0) (at 57.785 189.23 0)
-      (effects (font (size 1.27 1.27)) hide)
-    )
-    (property "Value" "+3.3V" (id 1) (at 57.785 182.245 0)
-      (effects (font (size 1.27 1.27)))
-    )
-    (property "Footprint" "" (id 2) (at 57.785 185.42 0)
-      (effects (font (size 1.27 1.27)) hide)
-    )
-    (property "Datasheet" "" (id 3) (at 57.785 185.42 0)
-      (effects (font (size 1.27 1.27)) hide)
-    )
-    (pin "1")
-  )
   (symbol (lib_id "Mechanical:MountingHole_Pad") (at 211.455 258.445 270) (unit 1)
     (in_bom yes) (on_board yes)
@@
       (reference "#PWR03") (unit 1) (value "GND") (footprint "")
     )
-    (path "/b8d9e664-27af-4ade-8670-64f712d84cb7"
-      (reference "#PWR04") (unit 1) (value "+3.3V") (footprint "")
-    )
     (path "/0150e33c-2f96-499e-885e-43103a792982"

Commit message: Update Training_Based.kicad_sch
Other:
- note added: "Recheck"
Changed lines of the file:
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@@
+    (effects (font (size 1.27 1.27)) (justify left bottom))
+  )
+  (text "Recheck" (at 34.29 111.76 0)
     (effects (font (size 1.27 1.27)) (justify left bottom))
   )

Commit message: WIP 650806-1532
Parts:
- added C (x3): C_Small, symbol Device:C_Small
- added D: D_Zener_Dual_CommonCathode_AAK_Split, symbol Device:D_Zener_Dual_CommonCathode_AAK_Split
Connections:
- net +3.3V: now also C.1
- net Analog_Input: now also D.3 (K)
- net GND: now also C.2, C.2, C.2, D.1 (A)
- net LDR_OUTPUT: now also C.1
- net Poten_voltage: now also C.1
Other:
- note added: "R = 100 ~ 500k OHM @100 OHM -> Vout = 3.26V @500k OHM -> Vout = 0.06V"
- note removed: "Recheck"
- moved on the sheet: J, R, RV, U

Commit message: Update Training_Based.kicad_sch
Parts:
- added R (x3): R_Small, symbol Device:R_Small
Connections:
- net +3.3V: now also R.1, R.1, R.1
- net A_Rotary: now also R.2
- net B_Rotary: now also R.2
- net S1_Rotary: now also R.2
Other:
- note added: "CAUTION! Vin_{MAX} = 35 V"
- moved on the sheet: J, R, SW

Commit message: Final Check
Connections:
- net +3.3V_ESP: no longer U.1 (3.3V)
- net +5V: now also J.8 (Pin_8), J.8 (Pin_8); no longer U.19 (5V)
- net EN_RST: no longer U.2 (EN_RST)
- net GND: now also J.1 (Pin_1), J.1 (Pin_1); no longer U.14 (GND), U.32 (GND), U.38 (GND)
- net GPI34: no longer U.5 (GPI34)
- net GPI35: no longer U.6 (GPI35)
- net GPI36: no longer U.3 (GPI36)
- net GPI39: no longer U.4 (GPI39)
- net GPIO0: no longer U.25 (GPIO0)
- net GPIO1: now also J.2 (Pin_2); no longer U.35 (GPIO1)
- net GPIO10: no longer U.17 (GPIO10)
- net GPIO11: no longer U.18 (GPIO11)
- net GPIO12: no longer U.13 (GPIO12)
- net GPIO13: now also J.7 (Pin_7); no longer U.15 (GPIO13)
- net GPIO14: now also J.6 (Pin_6); no longer U.12 (GPIO14)
- net GPIO15: no longer U.23 (GPIO15)
- net GPIO16: now also J.2 (Pin_2); no longer U.27 (GPIO16)
- net GPIO17: now also J.3 (Pin_3); no longer U.28 (GPIO17)
- net GPIO18: now also J.5 (Pin_5); no longer U.30 (GPIO18)
- net GPIO19: now also J.6 (Pin_6); no longer U.31 (GPIO19)
- net GPIO2: no longer U.24 (GPIO2)
- net GPIO21: now also J.5 (Pin_5); no longer U.33 (GPIO21)
- net GPIO22: now also J.4 (Pin_4); no longer U.36 (GPIO22)
- net GPIO23: now also J.7 (Pin_7); no longer U.37 (GPIO23)
- net GPIO25: no longer U.9 (GPIO25)
- net GPIO26: no longer U.10 (GPIO26)
- net GPIO27: no longer U.11 (GPIO27)
- net GPIO3: now also J.3 (Pin_3); no longer U.34 (GPIO3)
- net GPIO32: no longer U.7 (GPIO32)
- net GPIO33: no longer U.8 (GPIO33)
- net GPIO4: no longer U.26 (GPIO4)
- net GPIO5: now also J.4 (Pin_4); no longer U.29 (GPIO5)
- net GPIO6: no longer U.20 (GPIO6)
- net GPIO7: no longer U.21 (GPIO7)
- net GPIO8: no longer U.22 (GPIO8)
- net GPIO9: no longer U.16 (GPIO9)
Other:
- note added: "CAN RX"
- note added: "CAN TX"
- note added: "I2C SCL"
- note added: "I2C SDA"
- note added: "UART0 RX"
- note added: "UART0 TX"
- note added: "UART2 RX"
- note added: "UART2 TX"
- note added: "VSPI CLK"
- note added: "VSPI CS"
- note added: "VSPI MISO"
- note added: "VSPI MOSI"
- moved on the sheet: J, U

Commit message: Final 650807
Connections:
- net +3.3V_ESP: now also U.1 (3.3V)
- net +5V: now also U.19 (5V)
- net EN_RST: now also U.2 (EN_RST)
- net GND: now also U.14 (GND), U.32 (GND), U.38 (GND)
- net GPI34: now also U.5 (GPI34)
- net GPI35: now also U.6 (GPI35)
- net GPI36: now also U.3 (GPI36)
- net GPI39: now also U.4 (GPI39)
- net GPIO0: now also U.25 (GPIO0)
- net GPIO1: now also U.35 (GPIO1)
- net GPIO10: now also U.17 (GPIO10)
- net GPIO11: now also U.18 (GPIO11)
- net GPIO12: now also U.13 (GPIO12)
- net GPIO13: now also U.15 (GPIO13)
- net GPIO14: now also U.12 (GPIO14)
- net GPIO15: now also U.23 (GPIO15)
- net GPIO16: now also U.27 (GPIO16)
- net GPIO17: now also U.28 (GPIO17)
- net GPIO18: now also U.30 (GPIO18)
- net GPIO19: now also U.31 (GPIO19)
- net GPIO2: now also U.24 (GPIO2)
- net GPIO21: now also U.33 (GPIO21)
- net GPIO22: now also U.36 (GPIO22)
- net GPIO23: now also U.37 (GPIO23)
- net GPIO25: now also U.9 (GPIO25)
- net GPIO26: now also U.10 (GPIO26)
- net GPIO27: now also U.11 (GPIO27)
- net GPIO3: now also U.34 (GPIO3)
- net GPIO32: now also U.7 (GPIO32)
- net GPIO33: now also U.8 (GPIO33)
- net GPIO4: now also U.26 (GPIO4)
- net GPIO5: now also U.29 (GPIO5)
- net GPIO6: now also U.20 (GPIO6)
- net GPIO7: now also U.21 (GPIO7)
- net GPIO8: now also U.22 (GPIO8)
- net GPIO9: now also U.16 (GPIO9)
Other:
- note added: "V_{out}=0.6*(1+220k/49.9k)"
- note added: "V_{out}=0.6*(1+R_{1}/R_{2})"
- note added: "V_{out}=3.245V"
- moved on the sheet: U
Changed lines of the file:
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@@
     (effects (font (size 1.27 1.27)) (justify left bottom))
   )
-  (text "I2C SCL" (at 229.235 222.885 0)
+  (text "I2C SCL" (at 253.365 215.265 0)
+    (effects (font (size 1.27 1.27)) (justify left bottom))
+  )
+  (text "V_{out}=0.6*(1+R_{1}/R_{2})" (at 57.785 270.51 0)
     (effects (font (size 1.27 1.27)) (justify left bottom))
   )
@@
     (effects (font (size 1.27 1.27)) (justify left bottom))
   )
-  (text "UART2 TX" (at 229.235 183.515 0)
+  (text "UART2 TX" (at 229.87 183.515 0)
     (effects (font (size 1.27 1.27)) (justify left bottom))
   )
-  (text "CAN RX" (at 229.235 230.505 0)
+  (text "CAN RX" (at 245.11 194.31 0)
     (effects (font (size 1.27 1.27)) (justify left bottom))
   )
-  (text "I2C SDA" (at 229.235 225.425 0)
+  (text "I2C SDA" (at 253.365 217.805 0)
     (effects (font (size 1.27 1.27)) (justify left bottom))
   )
@@
     (effects (font (size 1.27 1.27)) (justify left bottom))
   )
-  (text "UART0 TX" (at 229.235 217.805 0)
+  (text "UART0 TX" (at 229.87 217.805 0)
     (effects (font (size 1.27 1.27)) (justify left bottom))
   )
@@
     (effects (font (size 1.27 1.27)) (justify left bottom))
   )
-  (text "UART0 RX" (at 229.235 220.345 0)
+  (text "UART0 RX" (at 229.87 220.345 0)
+    (effects (font (size 1.27 1.27)) (justify left bottom))
+  )
+  (text "UART2 RX" (at 229.87 186.055 0)
     (effects (font (size 1.27 1.27)) (justify left bottom))
   )
-  (text "UART2 RX" (at 229.235 186.055 0)
+  (text "V_{out}=0.6*(1+220k/49.9k)" (at 57.785 273.685 0)
     (effects (font (size 1.27 1.27)) (justify left bottom))
   )
-  (text "CAN TX" (at 229.235 227.965 0)
+  (text "CAN TX" (at 245.11 191.77 0)
     (effects (font (size 1.27 1.27)) (justify left bottom))
   )
@@
     (effects (font (size 1.27 1.27)) (justify left bottom))
   )
+  (text "V_{out}=3.245V" (at 57.785 276.86 0)
+    (effects (font (size 1.27 1.27)) (justify left bottom))
+  )
   (text "Servo Motor" (at 388.62 175.26 0)
     (effects (font (size 1.27 1.27)) (justify left bottom))
@@
       (effects (font (size 1.27 1.27)))
     )
-    (property "Value" "R_Small" (id 1) (at 261.62 247.015 90)
+    (property "Value" "R_Small" (id 1) (at 257.81 250.19 90)
       (effects (font (size 1.27 1.27)))
     )
@@
       (effects (font (size 1.27 1.27)))
     )
-    (property "Value" "R_Small" (id 1) (at 388.62 53.975 90)
+    (property "Value" "R_Small" (id 1) (at 384.81 56.515 90)
       (effects (font (size 1.27 1.27)))
     )
@@
       (effects (font (size 1.27 1.27)))
     )
-    (property "Value" "R_Small" (id 1) (at 353.06 53.975 90)
+    (property "Value" "R_Small" (id 1) (at 349.25 56.515 90)
       (effects (font (size 1.27 1.27)))
     )
@@
       (effects (font (size 1.27 1.27)))
     )
-    (property "Value" "R_Small" (id 1) (at 261.62 203.2 90)
+    (property "Value" "R_Small" (id 1) (at 257.81 206.375 90)
       (effects (font (size 1.27 1.27)))
     )
@@
     (pin "2")
   )
-  (symbol (lib_id "FP:esp32_38_pins-custom_library") (at 74.295 192.405 0) (mirror y) (unit 1)
+  (symbol (lib_id "FP:esp32_38_pins-custom_library") (at 74.295 192.405 0) (unit 1)
     (in_bom yes) (on_board yes)
     (default_instance (reference "U") (unit 1) (value "esp32_38_pins-custom_library") (footprint "esp32_lora_v2:esp32_devkitv4_38pin"))
-    (property "Reference" "U" (id 0) (at 65.405 183.515 0)
+    (property "Reference" "U" (id 0) (at 83.185 183.515 0)
       (effects (font (size 1.27 1.27)))
     )
-    (property "Value" "esp32_38_pins-custom_library" (id 1) (at 64.77 236.855 0)
+    (property "Value" "esp32_38_pins-custom_library" (id 1) (at 83.82 236.855 0)
       (effects (font (size 1.27 1.27)))
     )
-    (property "Footprint" "esp32_lora_v2:esp32_devkitv4_38pin" (id 2) (at 65.405 184.15 0)
+    (property "Footprint" "esp32_lora_v2:esp32_devkitv4_38pin" (id 2) (at 83.185 184.15 0)
       (effects (font (size 1.27 1.27)) hide)
     )
-    (property "Datasheet" "https://docs.espressif.com/projects/esp-idf/en/latest/get-started/get-started-devkitc.html" (id 3) (at 65.405 183.515 0)
+    (property "Datasheet" "https://docs.espressif.com/projects/esp-idf/en/latest/get-started/get-started-devkitc.html" (id 3) (at 83.185 183.515 0)
       (effects (font (size 1.27 1.27)) hide)
     )
@@
     )
     (path "/4366fa4a-643c-428b-ac2e-93563289719d"
-      (reference "P1") (unit 1) (value "K1") (footprint "Connector_Phoenix_MC:PhoenixContact_MC_1,5_3-G-3.5_1x03_P3.50mm_Horizontal")
+      (reference "P1") (unit 1) (value "K1") (footprint "TerminalBlock_MetzConnect:TerminalBlock_MetzConnect_Type059_RT06303HBWC_1x03_P3.50mm_Horizontal")
     )
     (path "/52721ab9-58f8-4ab1-983f-34277bf4e325"
-      (reference "P2") (unit 1) (value "K2") (footprint "Connector_Phoenix_MC:PhoenixContact_MC_1,5_3-G-3.5_1x03_P3.50mm_Horizontal")
+      (reference "P2") (unit 1) (value "K2") (footprint "TerminalBlock_MetzConnect:TerminalBlock_MetzConnect_Type059_RT06303HBWC_1x03_P3.50mm_Horizontal")
     )
     (path "/d24eb234-3298-4278-83ce-8e628b7976ab"
@@
     )
     (path "/e5715323-0243-4641-9e19-dde35912844b"
-      (reference "P5") (unit 1) (value "Voltage Input") (footprint "Connector_Phoenix_MC:PhoenixContact_MC_1,5_2-G-3.5_1x02_P3.50mm_Horizontal")
+      (reference "P5") (unit 1) (value "Voltage Input") (footprint "TerminalBlock_MetzConnect:TerminalBlock_MetzConnect_Type059_RT06302HBWC_1x02_P3.50mm_Horizontal")
     )
     (path "/ffbc64ff-e590-493d-b60f-cf4b737cad6e"
@@
     )
     (path "/8fc30915-4256-4cd2-958e-381089100f6c"
-      (reference "R19") (unit 1) (value "10k") (footprint "Resistor_SMD:R_0603_1608Metric")
+      (reference "R19") (unit 1) (value "4.7k") (footprint "Resistor_SMD:R_0603_1608Metric")
     )
     (path "/31aee95c-8482-489c-baf0-df95c1bb282b"
-      (reference "R20") (unit 1) (value "10k") (footprint "Resistor_SMD:R_0603_1608Metric")
+      (reference "R20") (unit 1) (value "4.7k") (footprint "Resistor_SMD:R_0603_1608Metric")
     )
     (path "/713c97ea-63b6-41f3-8697-8f30c3dd5553"
-      (reference "R21") (unit 1) (value "10k") (footprint "Resistor_SMD:R_0603_1608Metric")
+      (reference "R21") (unit 1) (value "4.7k") (footprint "Resistor_SMD:R_0603_1608Metric")
     )
     (path "/56d8adc8-e967-4680-8122-abb7a121c81e"
-      (reference "R22") (unit 1) (value "10k") (footprint "Resistor_SMD:R_0603_1608Metric")
+      (reference "R22") (unit 1) (value "4.7k") (footprint "Resistor_SMD:R_0603_1608Metric")
     )
     (path "/1b3c17bd-0c66-4002-9029-d76f74818636"

Commit message: Update Training_Based.kicad_sch
Connections:
- net +3.3V: now also D.2 (A), D.2 (A)
- net +5V: no longer D.2 (A), D.2 (A)
Other:
- note added: "OK"
Changed lines of the file:
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@@
     (effects (font (size 1.27 1.27)) (justify left bottom))
   )
+  (text "OK" (at 148.59 59.055 0)
+    (effects (font (size 1.27 1.27)) (justify left bottom))
+  )
+  (text "OK" (at 388.62 50.8 0)
+    (effects (font (size 1.27 1.27)) (justify left bottom))
+  )
+  (text "OK" (at 93.98 59.055 0)
+    (effects (font (size 1.27 1.27)) (justify left bottom))
+  )
   (text "CAN RX" (at 245.11 194.31 0)
     (effects (font (size 1.27 1.27)) (justify left bottom))
   )
+  (text "OK" (at 313.055 45.72 0)
+    (effects (font (size 1.27 1.27)) (justify left bottom))
+  )
   (text "I2C SDA" (at 253.365 217.805 0)
     (effects (font (size 1.27 1.27)) (justify left bottom))
   )
+  (text "OK" (at 46.99 60.96 0)
+    (effects (font (size 1.27 1.27)) (justify left bottom))
+  )
+  (text "OK" (at 313.69 57.15 0)
+    (effects (font (size 1.27 1.27)) (justify left bottom))
+  )
   (text "7 Segment 4 Digit TM1637" (at 352.425 17.145 0)
     (effects (font (size 1.27 1.27)) (justify left bottom))
@@
     (effects (font (size 1.27 1.27)) (justify left bottom))
   )
+  (text "OK" (at 172.085 53.34 0)
+    (effects (font (size 1.27 1.27)) (justify left bottom))
+  )
   (text "UART0 TX" (at 229.87 217.805 0)
     (effects (font (size 1.27 1.27)) (justify left bottom))
   )
+  (text "OK" (at 167.005 36.195 0)
+    (effects (font (size 1.27 1.27)) (justify left bottom))
+  )
   (text "R = 100 ~ 500k OHM\n@100 OHM  -> Vout = 3.26V\n@500k OHM -> Vout = 0.06V\n"
     (at 82.55 83.82 0)
@@
     (effects (font (size 1.27 1.27)) (justify left bottom))
   )
+  (text "OK" (at 398.78 58.42 0)
+    (effects (font (size 1.27 1.27)) (justify left bottom))
+  )
   (text "UART0 RX" (at 229.87 220.345 0)
     (effects (font (size 1.27 1.27)) (justify left bottom))
   )
+  (text "OK" (at 130.81 36.195 0)
+    (effects (font (size 1.27 1.27)) (justify left bottom))
+  )
+  (text "OK" (at 363.855 58.42 0)
+    (effects (font (size 1.27 1.27)) (justify left bottom))
+  )
   (text "UART2 RX" (at 229.87 186.055 0)
     (effects (font (size 1.27 1.27)) (justify left bottom))
   )
+  (text "OK" (at 134.62 53.34 0)
+    (effects (font (size 1.27 1.27)) (justify left bottom))
+  )
   (text "V_{out}=0.6*(1+220k/49.9k)" (at 57.785 273.685 0)
     (effects (font (size 1.27 1.27)) (justify left bottom))
@@
     (effects (font (size 1.27 1.27)) (justify left bottom))
   )
+  (text "OK" (at 48.895 48.895 0)
+    (effects (font (size 1.27 1.27)) (justify left bottom))
+  )
   (text "ESP32 38 PIN" (at 129.54 176.53 0)
     (effects (font (size 1.27 1.27)) (justify left bottom))
   )
+  (text "OK" (at 97.79 40.005 0)
+    (effects (font (size 1.27 1.27)) (justify left bottom))
+  )
   (label "GPIO15" (at 98.425 225.425 0) (fields_autoplaced)
     (effects (font (size 1.27 1.27)) (justify left bottom))
@@
     (pin "1")
   )
+  (symbol (lib_id "power:+3.3V") (at 137.16 123.825 0) (unit 1)
+    (in_bom yes) (on_board yes) (fields_autoplaced)
+    (default_instance (reference "#PWR") (unit 1) (value "+3.3V") (footprint ""))
+    (property "Reference" "#PWR" (id 0) (at 137.16 127.635 0)
+      (effects (font (size 1.27 1.27)) hide)
+    )
+    (property "Value" "+3.3V" (id 1) (at 137.16 120.65 0)
+      (effects (font (size 1.27 1.27)))
+    )
+    (property "Footprint" "" (id 2) (at 137.16 123.825 0)
+      (effects (font (size 1.27 1.27)) hide)
+    )
+    (property "Datasheet" "" (id 3) (at 137.16 123.825 0)
+      (effects (font (size 1.27 1.27)) hide)
+    )
+    (pin "1")
+  )
   (symbol (lib_id "Device:LED") (at 315.595 139.065 90) (unit 1)
     (in_bom yes) (on_board yes)
@@
     (in_bom yes) (on_board yes)
     (default_instance (reference "U") (unit 1) (value "HC-SR04") (footprint ""))
-    (property "Reference" "U" (id 0) (at 99.695 28.575 0)
+    (property "Reference" "U" (id 0) (at 95.885 24.13 0)
       (effects (font (size 1.524 1.524)) (justify left))
     )
-    (property "Value" "HC-SR04" (id 1) (at 85.725 26.67 0)
+    (property "Value" "HC-SR04" (id 1) (at 88.265 26.67 0)
       (effects (font (size 1.524 1.524)) (justify left))
     )
@@
     (in_bom yes) (on_board yes)
     (default_instance (reference "TH") (unit 1) (value "DHT22_Temperature_Humidity") (footprint ""))
-    (property "Reference" "TH" (id 0) (at 50.8 30.48 0)
+    (property "Reference" "TH" (id 0) (at 45.72 25.4 0)
       (effects (font (size 1.524 1.524)) (justify left))
     )
-    (property "Value" "DHT22_Temperature_Humidity" (id 1) (at 24.13 26.67 0)
+    (property "Value" "DHT22_Temperature_Humidity" (id 1) (at 24.13 27.94 0)
       (effects (font (size 1.524 1.524)) (justify left))
     )
@@
     (pin "2")
   )
+  (symbol (lib_id "power:+3.3V") (at 137.16 146.685 0) (unit 1)
+    (in_bom yes) (on_board yes) (fields_autoplaced)
+    (default_instance (reference "#PWR") (unit 1) (value "+3.3V") (footprint ""))
+    (property "Reference" "#PWR" (id 0) (at 137.16 150.495 0)
+      (effects (font (size 1.27 1.27)) hide)
+    )
+    (property "Value" "+3.3V" (id 1) (at 137.16 143.51 0)
+      (effects (font (size 1.27 1.27)))
+    )
+    (property "Footprint" "" (id 2) (at 137.16 146.685 0)
+      (effects (font (size 1.27 1.27)) hide)
+    )
+    (property "Datasheet" "" (id 3) (at 137.16 146.685 0)
+      (effects (font (size 1.27 1.27)) hide)
+    )
+    (pin "1")
+  )
   (symbol (lib_id "Transistor_BJT:BC817") (at 167.005 46.99 0) (unit 1)
     (in_bom yes) (on_board yes) (fields_autoplaced)
@@
     (pin "1")
   )
-  (symbol (lib_id "power:+5V") (at 137.16 123.825 0) (unit 1)
-    (in_bom yes) (on_board yes) (fields_autoplaced)
-    (default_instance (reference "#PWR") (unit 1) (value "+5V") (footprint ""))
-    (property "Reference" "#PWR" (id 0) (at 137.16 127.635 0)
-      (effects (font (size 1.27 1.27)) hide)
-    )
-    (property "Value" "+5V" (id 1) (at 137.16 120.015 0)
-      (effects (font (size 1.27 1.27)))
-    )
-    (property "Footprint" "" (id 2) (at 137.16 123.825 0)
-      (effects (font (size 1.27 1.27)) hide)
-    )
-    (property "Datasheet" "" (id 3) (at 137.16 123.825 0)
-      (effects (font (size 1.27 1.27)) hide)
-    )
-    (pin "1")
-  )
   (symbol (lib_id "power:GND") (at 75.565 94.615 0) (unit 1)
     (in_bom yes) (on_board yes) (fields_autoplaced)
@@
     (pin "3")
   )
-  (symbol (lib_id "power:+5V") (at 137.16 146.685 0) (unit 1)
-    (in_bom yes) (on_board yes) (fields_autoplaced)
-    (default_instance (reference "#PWR") (unit 1) (value "+5V") (footprint ""))
-    (property "Reference" "#PWR" (id 0) (at 137.16 150.495 0)
-      (effects (font (size 1.27 1.27)) hide)
-    )
-    (property "Value" "+5V" (id 1) (at 137.16 142.875 0)
-      (effects (font (size 1.27 1.27)))
-    )
-    (property "Footprint" "" (id 2) (at 137.16 146.685 0)
-      (effects (font (size 1.27 1.27)) hide)
-    )
-    (property "Datasheet" "" (id 3) (at 137.16 146.685 0)
-      (effects (font (size 1.27 1.27)) hide)
-    )
-    (pin "1")
-  )
   (symbol (lib_id "Device:R_Small") (at 349.25 146.05 0) (unit 1)
     (in_bom yes) (on_board yes)
@@
       (reference "#PWR046") (unit 1) (value "GND") (footprint "")
     )
-    (path "/c6388885-836e-4bf9-9798-3cb11d0d97a7"
-      (reference "#PWR047") (unit 1) (value "+5V") (footprint "")
+    (path "/1d2731cd-94f0-460a-b914-6d09a0579550"
+      (reference "#PWR047") (unit 1) (value "+3.3V") (footprint "")
     )
     (path "/a2429c51-bdfa-4091-a4c6-e2bd28712fe6"
@@
       (reference "#PWR051") (unit 1) (value "+3.3V") (footprint "")
     )
-    (path "/d7c2c74f-edac-4f56-a934-1f68f35d847d"
-      (reference "#PWR052") (unit 1) (value "+5V") (footprint "")
+    (path "/b1e37e12-5935-4335-b232-a8c0eeba2028"
+      (reference "#PWR052") (unit 1) (value "+3.3V") (footprint "")
     )
     (path "/82b4e88d-dbac-4c55-99c2-0add9da3f4c8"
