File: Training_Based.kicad_pcb (KiCad board)
At the start: 2 copper layers, 210 x 140 mm, 133 parts, among them J1 ESP32_LEFT_A, J10 7 Segment Digit, J11 7 Segment Common, J12 SERVO MOTOR, J13 SERVO 1, J14 SERVO 2, J15 OPTO ISOLATOR, J16 OPTO, J17 SWITCH, J18 Analog Input, J19 USB_B_Mini, J2 ESP32_LEFT_B, J20 +5V, J21 +3.3V, J22 GND, J23 Conn_01x08, J24 Conn_01x08, J3 ESP32_RIGHT_A, J4 ESP32_RIGHT_B, J5 LED x8, J6 TEMP-HUMID, J7 Ultrasonic, J8 Buzzer, J9 RELAY, K1 FINDER-36.11, K2 FINDER-36.11, P1 K1, P2 K2, P3 OPTO INPUT 1, P4 OPTO INPUT 2, P5 Voltage Input, Q1 BC817, Q10 BC817, Q11 BC817, Q12 BC817, Q13 BC817, Q14 BC817, Q2 BC817, Q3 BC817, Q4 BC817, Q5 BC817, Q6 BC817, Q7 BC817, Q8 BC817, Q9 BC817, SW1 RotaryEncoder_Switch, SW2 SW_Push, SW3 SW_Push, U1 HC-SR04, U2 Protoboard, U3 esp32_38_pins-custom_library, U4 DC56-11SURKWA, U5 LTV-827, U6 TSOP382xx, U7 SY8089AAAC(SOT23-5)

Commit message: WIP 650806-1532
Parts:
- added C6: 1nF, Capacitor_SMD:C_0603_1608Metric, F.Cu at (61.9, 74.3)
- added C7: 0.1uF, Capacitor_SMD:C_0603_1608Metric, F.Cu at (76.8, 58.8)
- added C8: 1nF, Capacitor_SMD:C_0603_1608Metric, F.Cu at (48.6, 107.3)
- added D3: BZX84C3V3LT1G, Package_TO_SOT_SMD:SOT-323_SC-70, F.Cu at (48.0, 115.8)
- added G***: LOGO, Training_Based:KMITL, F.Cu at (203.8, 137.0)
- added R48: 10k, Resistor_SMD:R_0603_1608Metric, F.Cu at (93.8, 119.1)
- added R49: 10k, Resistor_SMD:R_0603_1608Metric, F.Cu at (93.8, 121.6)
- added R50: 10k, Resistor_SMD:R_0603_1608Metric, F.Cu at (93.8, 116.5)
- R43: value R_Small -> 100k
- R44: value R_Small -> 10k
- moved Q12 7.52 mm to (183.1, 65.3)
- moved R20 7.22 mm to (180.3, 65.3), turned to 90 degrees
- moved Q11 3.95 mm to (183.1, 83.4)
- moved R19 3.93 mm to (180.3, 83.4)
- moved J14 2.95 mm to (212.9, 106.3)
- moved J13 2.95 mm to (212.9, 96.6)
- moved R32 2.78 mm to (185.8, 65.3)
- moved J18 2.40 mm to (54.4, 106.5)
- moved D2 1.20 mm to (188.1, 65.2)
- moved R31 0.34 mm to (185.8, 83.4)
- moved U1 0.20 mm to (63.0, 32.2)
- turned LED9 to 90 degrees
Routing:
- net +5V: track 152.3 -> 0.00 mm
- net /S_F: track 46.2 -> 0.00 mm, vias 1 -> 0
- net /S_B: track 38.3 -> 0.00 mm
- net /S_A: track 38.1 -> 0.00 mm
- net /S_G: track 28.6 -> 0.00 mm
- net /S_DP: track 25.2 -> 0.00 mm
- net /S_C: track 23.5 -> 0.00 mm, vias 1 -> 0
- net +3.3V: track 22.9 -> 0.00 mm
- net Net-(Q13-B): track 21.3 -> 0.00 mm
- net /S_E: track 20.9 -> 0.00 mm
- net Net-(Q14-B): track 19.3 -> 0.00 mm
- net /GPIO23: track 17.1 -> 0.00 mm
- net /GPIO22: track 17.1 -> 0.00 mm
- net /GPIO1: track 17.1 -> 0.00 mm
- net /GPIO8: track 17.1 -> 0.00 mm
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Other:
- board text added: "(c) 2022"
- board text added: "CAUTION! Vin_{MAX} = 35V."
- board text added: "DIGITAL INPUT"
- board text added: "PWM"
- board text added: "SERVO 1"
- board text added: "SERVO 2"
- board text removed: "SERVO MOTOR 1"
- board text removed: "SERVO MOTOR 2"
- board text removed: "Servo 1"
- board text removed: "Servo 2"
- board text removed: "ULTRASONIC SENSOR"

Commit message: Final Check
Parts:
- added G***: LOGO, Training_Based:SIET_15x15, F.Cu at (188.3, 136.9)
- P3, P4: footprint Connector_Phoenix_MC:PhoenixContact_MC_1,5_2-G-3.5_1x02_P3.50mm_Horizontal -> TerminalBlock_MetzConnect:TerminalBlock_MetzConnect_Type059_RT06302HBWC_1x02_P3.50mm_Horizontal
- moved C6 9.14 mm to (66.5, 66.4), turned to 90 degrees
- moved R38 8.83 mm to (68.1, 66.4), turned to -90 degrees
- moved G*** 8.47 mm to (212.3, 136.9)
- moved F1 3.82 mm to (34.4, 144.6), turned to 90 degrees
- moved C1 1.87 mm to (37.7, 145.9)
- moved C2 1.87 mm to (43.9, 150.4)
- moved L1 1.87 mm to (45.5, 146.1)
- moved R46 1.87 mm to (43.9, 148.8)
- moved R47 1.87 mm to (40.8, 148.8)
- moved U7 1.87 mm to (41.2, 146.0)
- moved C4 1.87 mm to (48.5, 146.0)
- moved P4 0.48 mm to (30.1, 88.4)
- moved P3 0.43 mm to (30.1, 78.4)
- turned R17 to 180 degrees
- turned R32 to 90 degrees
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Connections:
- J23 pad 1: unconnected-(J23-Pin_1) -> GND
- J23 pad 2: unconnected-(J23-Pin_2) -> /GPIO1
- J23 pad 3: unconnected-(J23-Pin_3) -> /GPIO3
- J23 pad 4: unconnected-(J23-Pin_4) -> /GPIO22
- J23 pad 5: unconnected-(J23-Pin_5) -> /GPIO21
- J23 pad 6: unconnected-(J23-Pin_6) -> /GPIO14
- J23 pad 7: unconnected-(J23-Pin_7) -> /GPIO13
- J23 pad 8: unconnected-(J23-Pin_8) -> +5V
- J24 pad 1: unconnected-(J24-Pin_1) -> GND
- J24 pad 2: unconnected-(J24-Pin_2) -> /GPIO16
- J24 pad 3: unconnected-(J24-Pin_3) -> /GPIO17
- J24 pad 4: unconnected-(J24-Pin_4) -> /GPIO5
- J24 pad 5: unconnected-(J24-Pin_5) -> /GPIO18
- J24 pad 6: unconnected-(J24-Pin_6) -> /GPIO19
- J24 pad 7: unconnected-(J24-Pin_7) -> /GPIO23
- J24 pad 8: unconnected-(J24-Pin_8) -> +5V
- U3 pad 1: /+3.3V_ESP -> unconnected-(U3-3.3V)
- U3 pad 10: /GPIO26 -> unconnected-(U3-GPIO26)
- U3 pad 11: /GPIO27 -> unconnected-(U3-GPIO27)
- U3 pad 12: /GPIO14 -> unconnected-(U3-GPIO14)
- U3 pad 13: /GPIO12 -> unconnected-(U3-GPIO12)
- U3 pad 14: GND -> unconnected-(U3-GND)_1
- U3 pad 15: /GPIO13 -> unconnected-(U3-GPIO13)
- U3 pad 16: /GPIO9 -> unconnected-(U3-GPIO9)
- U3 pad 17: /GPIO10 -> unconnected-(U3-GPIO10)
- U3 pad 19: +5V -> unconnected-(U3-5V)
- U3 pad 2: /EN_RST -> unconnected-(U3-EN_RST)
- U3 pad 20: /GPIO6 -> unconnected-(U3-GPIO6)
- U3 pad 21: /GPIO7 -> unconnected-(U3-GPIO7)
- U3 pad 22: /GPIO8 -> unconnected-(U3-GPIO8)
- U3 pad 23: /GPIO15 -> unconnected-(U3-GPIO15)
- U3 pad 24: /GPIO2 -> unconnected-(U3-GPIO2)
- U3 pad 25: /GPIO0 -> unconnected-(U3-GPIO0)
- U3 pad 26: /GPIO4 -> unconnected-(U3-GPIO4)
- U3 pad 27: /GPIO16 -> unconnected-(U3-GPIO16)
- U3 pad 28: /GPIO17 -> unconnected-(U3-GPIO17)
- U3 pad 29: /GPIO5 -> unconnected-(U3-GPIO5)
- U3 pad 3: /GPI36 -> unconnected-(U3-GPI36)
- U3 pad 30: /GPIO18 -> unconnected-(U3-GPIO18)
- U3 pad 31: /GPIO19 -> unconnected-(U3-GPIO19)
- U3 pad 32: GND -> unconnected-(U3-GND)_2
- U3 pad 33: /GPIO21 -> unconnected-(U3-GPIO21)
- U3 pad 34: /GPIO3 -> unconnected-(U3-GPIO3)
- U3 pad 35: /GPIO1 -> unconnected-(U3-GPIO1)
- U3 pad 36: /GPIO22 -> unconnected-(U3-GPIO22)
- U3 pad 37: /GPIO23 -> unconnected-(U3-GPIO23)
- U3 pad 38: GND -> unconnected-(U3-GND)
- U3 pad 4: /GPI39 -> unconnected-(U3-GPI39)
- U3 pad 5: /GPI34 -> unconnected-(U3-GPI34)
- U3 pad 6: /GPI35 -> unconnected-(U3-GPI35)
- U3 pad 7: /GPIO32 -> unconnected-(U3-GPIO32)
- U3 pad 8: /GPIO33 -> unconnected-(U3-GPIO33)
- U3 pad 9: /GPIO25 -> unconnected-(U3-GPIO25)
Routing:
- net +5V: track 0.00 -> 784.2 mm, vias 0 -> 8
- net +3.3V: track 0.00 -> 138.5 mm, vias 0 -> 3
- net /GPIO13: track 0.00 -> 119.7 mm
- net /GPIO14: track 0.00 -> 118.3 mm
- net /GPIO23: track 0.00 -> 97.7 mm, vias 0 -> 1
- net /GPIO19: track 0.00 -> 76.4 mm
- net /GPIO18: track 0.00 -> 72.0 mm
- net /GPIO5: track 0.00 -> 67.1 mm
- net GND: track 0.00 -> 63.2 mm, vias 0 -> 73
- net /GPIO17: track 0.00 -> 62.4 mm
- net /GPIO16: track 0.00 -> 57.3 mm
- net /GPIO21: track 0.00 -> 51.0 mm
- net /GPIO22: track 0.00 -> 47.1 mm
- net /GPIO3: track 0.00 -> 43.4 mm
- net /S_B: track 0.00 -> 43.4 mm, vias 0 -> 2
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- added copper zone on B.Cu, net GND
Other:
- board text added: "+"
- board text added: "-"
- board text added: "locked"
- board text removed: "(c) 2022"
- board text removed: "+3.3V"
- board text removed: "+5.0V"
- board text removed: "1"
- board text removed: "2"
- board text removed: "3"
- board text removed: "4"
- board text removed: "5"
- board text removed: "6"
- board text removed: "7"
- board text removed: "7SEGMENT LED"
- board text removed: "8"
- board text removed: "ANALOG INPUT"
- board text removed: "BREAKOUT AREA"
- board text removed: "BUZZER"
- board text removed: "BZ1"
- board text removed: "BZ2"
- board text removed: "CAUTION! Vin_{MAX} = 35V."
- board text removed: "COM"
- board text removed: "D1"
- board text removed: "D2"
- board text removed: "DATA"
- board text removed: "DIGITAL INPUT"
- board text removed: "Echo"
- board text removed: "LDR"
- board text removed: "LEDs"
- board text removed: "NC"
- board text removed: "NO"
- board text removed: "OPTO Electronic"
- board text removed: "OPTO IN 1"
- board text removed: "OPTO IN 2"
- board text removed: "OPTO INPUT 1"
- board text removed: "OPTO INPUT 2"
- board text removed: "PIR"
- board text removed: "POWER SUPPLY"
- board text removed: "PUSH BT1"
- board text removed: "PUSH BT2"
- board text removed: "PWM"
- board text removed: "RELAY OUTPUT"
- board text removed: "ROTARY"
- board text removed: "RY1"
- board text removed: "RY2"
- board text removed: "Rotary A"
- board text removed: "Rotary B"
- board text removed: "Rotary S1"
- board text removed: "SERVO 1"
- board text removed: "SERVO 2"
- board text removed: "SERVO MOTOR"
- board text removed: "TEMP/HUMID"
- board text removed: "Trig"
- board text removed: "V-"
- board text removed: "VOLUME"
- board text removed: "X"
- board text removed: "a"
- board text removed: "b"
- board text removed: "c"
- board text removed: "d"
- board text removed: "dp"
- board text removed: "e"
- board text removed: "f"
- board text removed: "g"

Commit message: Final 650807
Parts:
- P1, P2: footprint Connector_Phoenix_MC:PhoenixContact_MC_1,5_3-G-3.5_1x03_P3.50mm_Horizontal -> TerminalBlock_MetzConnect:TerminalBlock_MetzConnect_Type059_RT06303HBWC_1x03_P3.50mm_Horizontal
- P5: footprint Connector_Phoenix_MC:PhoenixContact_MC_1,5_2-G-3.5_1x02_P3.50mm_Horizontal -> TerminalBlock_MetzConnect:TerminalBlock_MetzConnect_Type059_RT06302HBWC_1x02_P3.50mm_Horizontal
- renumbered G*** to GKMITLLOGO, G*** to GSIETLOGO
Connections:
- U3 pad 1: unconnected-(U3-3.3V) -> /+3.3V_ESP
- U3 pad 10: unconnected-(U3-GPIO26) -> /GPIO26
- U3 pad 11: unconnected-(U3-GPIO27) -> /GPIO27
- U3 pad 12: unconnected-(U3-GPIO14) -> /GPIO14
- U3 pad 13: unconnected-(U3-GPIO12) -> /GPIO12
- U3 pad 14: unconnected-(U3-GND)_1 -> GND
- U3 pad 15: unconnected-(U3-GPIO13) -> /GPIO13
- U3 pad 16: unconnected-(U3-GPIO9) -> /GPIO9
- U3 pad 17: unconnected-(U3-GPIO10) -> /GPIO10
- U3 pad 19: unconnected-(U3-5V) -> +5V
- U3 pad 2: unconnected-(U3-EN_RST) -> /EN_RST
- U3 pad 20: unconnected-(U3-GPIO6) -> /GPIO6
- U3 pad 21: unconnected-(U3-GPIO7) -> /GPIO7
- U3 pad 22: unconnected-(U3-GPIO8) -> /GPIO8
- U3 pad 23: unconnected-(U3-GPIO15) -> /GPIO15
- U3 pad 24: unconnected-(U3-GPIO2) -> /GPIO2
- U3 pad 25: unconnected-(U3-GPIO0) -> /GPIO0
- U3 pad 26: unconnected-(U3-GPIO4) -> /GPIO4
- U3 pad 27: unconnected-(U3-GPIO16) -> /GPIO16
- U3 pad 28: unconnected-(U3-GPIO17) -> /GPIO17
- U3 pad 29: unconnected-(U3-GPIO5) -> /GPIO5
- U3 pad 3: unconnected-(U3-GPI36) -> /GPI36
- U3 pad 30: unconnected-(U3-GPIO18) -> /GPIO18
- U3 pad 31: unconnected-(U3-GPIO19) -> /GPIO19
- U3 pad 32: unconnected-(U3-GND)_2 -> GND
- U3 pad 33: unconnected-(U3-GPIO21) -> /GPIO21
- U3 pad 34: unconnected-(U3-GPIO3) -> /GPIO3
- U3 pad 35: unconnected-(U3-GPIO1) -> /GPIO1
- U3 pad 36: unconnected-(U3-GPIO22) -> /GPIO22
- U3 pad 37: unconnected-(U3-GPIO23) -> /GPIO23
- U3 pad 38: unconnected-(U3-GND) -> GND
- U3 pad 4: unconnected-(U3-GPI39) -> /GPI39
- U3 pad 5: unconnected-(U3-GPI34) -> /GPI34
- U3 pad 6: unconnected-(U3-GPI35) -> /GPI35
- U3 pad 7: unconnected-(U3-GPIO32) -> /GPIO32
- U3 pad 8: unconnected-(U3-GPIO33) -> /GPIO33
- U3 pad 9: unconnected-(U3-GPIO25) -> /GPIO25
Routing:
- net +3.3V: track 138.5 -> 333.7 mm, vias 3 -> 5
- net +5V: track 784.2 -> 789.1 mm, vias 8 -> 9
- net /S_B: track 43.4 -> 45.0 mm, vias 2 -> 3
- net /S_A: track 42.6 -> 43.7 mm, vias 2 -> 3
- net GND: vias 73 -> 83
Other:
- board text added: "EN_RST"
- board text removed: "EN-RST"
- board text removed: "V+"

Commit message: Update Training_Based.kicad_pcb
Routing:
- net GND: vias 83 -> 124

Commit message: Update Training_Based.kicad_pcb
Parts:
- R19, R20, R21, R22: value 10k -> 4.7k
Connections:
- LED11 pad 2: +5V -> +3.3V
- LED12 pad 2: +5V -> +3.3V
Routing:
- net +5V: track 789.1 -> 747.9 mm, vias 9 -> 7
- net +3.3V: track 333.7 -> 339.1 mm
